File: Learn_KiCad.kicad_sch (KiCad schematic)
At the start: 41 parts, among them J1 USB_C_Receptacle_USB2.0, J2 TC2030, J3 Conn_01x04_Pin, J4 Conn_Coaxial, SW1 SW_Push, U1 MIC5365-3.3YD5, U2 USBLC6-2SC6, U3 STM32WB55CEU6, X1 32kHz768, X2 32MHz

Commit message: 2024-01-09 5:03
Parts:
- C16: Distributor Link (none) -> https://www.mouser.ca/ProductDetail/Murata-Electronics/GRM1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; Manufacturer (none) -> Murata Electronics; Manufacturer Part Number (none) -> GRM1555C1HR30WA01D
- C17, C18: Distributor Link (none) -> https://www.mouser.ca/ProductDetail/KYOCERA-AVX/04025A100JA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; Manufacturer (none) -> KYOCERA AVX; Manufacturer Part Number (none) -> 04025A100JAT4A
- D1: Distributor Link (none) -> https://www.mouser.ca/ProductDetail/Wurth-Elektronik/150040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; Manufacturer (none) -> Wurth Elektronik; Manufacturer Part Number (none) -> 150040RS73240
- FLT1: Distributor Link (none) -> https://www.mouser.ca/ProductDetail/TDK/DLF162500LT-5028A1?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; Manufacturer (none) -> TDK; Manufacturer Part Number (none) -> DLF162500LT-5028A1
- J1: Distributor Link (none) -> https://www.mouser.ca/ProductDetail/GCT/USB4105-GF-A?qs=KUo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; Manufacturer (none) -> GCT; Manufacturer Part Number (none) -> USB4105-GF-A
- J3: Distributor Link (none) -> https://www.mouser.ca/ProductDetail/Molex/53048-0410?qs=359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; Manufacturer (none) -> Molex; Manufacturer Part Number (none) -> 53048-0410
- J4: Distributor Link (none) -> https://www.mouser.ca/ProductDetail/Hirose-Connector/U.FL-R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; Manufacturer (none) -> Hirose Connector; Manufacturer Part Number (none) -> U.FL-R-SMT(01)
- L1: Distributor Link (none) -> https://www.mouser.ca/ProductDetail/Murata-Electronics/LQG1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; Manufacturer (none) -> Murata Electronics; Manufacturer Part Number (none) -> LQG15WZ10NJ02D
- L2: Distributor Link (none) -> https://www.mouser.ca/ProductDetail/Murata-Electronics/LQM2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; Manufacturer (none) -> Murata Electronics; Manufacturer Part Number (none) -> LQM21DH100M70L
- L3: Distributor Link (none) -> https://www.mouser.ca/ProductDetail/Murata-Electronics/LQG1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; Manufacturer (none) -> Murata Electronics; Manufacturer Part Number (none) -> LQG15HS2N7S02D
- R1, R2, R6: Distributor Link (none) -> https://www.mouser.ca/ProductDetail/YAGEO/RC0402FR-075K1L?q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; Manufacturer (none) -> YAGEO; Manufacturer Part Number (none) -> RC0402FR-075K1L
- R3, R4, R5, R7: Distributor Link (none) -> https://www.mouser.ca/ProductDetail/YAGEO/RC0402FR-07220RL?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; Manufacturer (none) -> YAGEO; Manufacturer Part Number (none) -> RC0402FR-07220RL
- SW1: Distributor Link (none) -> https://www.mouser.ca/ProductDetail/CK/RS282G05A3SMRT?qs=Gu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; Manufacturer (none) -> C&K; Manufacturer Part Number (none) -> RS282G05A3SMRT
- U1: Distributor Link (none) -> https://www.mouser.ca/ProductDetail/Microchip-Technology/MI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; Manufacturer (none) -> Microchip Technology; Manufacturer Part Number (none) -> MIC5365-3.3YD5-TR
- U2: Distributor Link (none) -> https://www.mouser.ca/ProductDetail/STMicroelectronics/USBL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; Manufacturer (none) -> STMicroelectronics; Manufacturer Part Number (none) -> SBLC6-2SC6
- U3: Distributor Link (none) -> https://www.mouser.ca/ProductDetail/STMicroelectronics/STM3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; Manufacturer (none) -> STMicroelectronics; Manufacturer Part Number (none) -> STM32WB55CEU6
Connections:
- removed net USER_CC1: J1.A5 (CC1), J1.A6 (D+), J1.A7 (D-), J1.B6 (D+), J1.B7 (D-), R2.1, U2.1 (I/O1), U2.3 (I/O2)
- net USER_CC2 renamed USBC_CC2
- new net USBC_CC1: J1.A5 (CC1), R2.1
- new net USBC_D+: J1.A6 (D+), J1.B6 (D+), U2.3 (I/O2)
- new net USBC_D-: J1.A7 (D-), J1.B7 (D-), U2.1 (I/O1)

Commit message: 2024-01-13 22:28
Connections:
- net BSW: now reaches R7.2, SW1.1
Changed lines of the file:
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@@
+    (effects (font (size 0.5 0.5)) (justify left bottom))
+  )
+  (label "BSW" (at 229.87 133.35 0) (fields_autoplaced)
     (effects (font (size 0.5 0.5)) (justify left bottom))
   )

Commit message: 2024-02-01 8:33am
Parts:
- added FM1, FM2, FM3: Fiducial, Fiducial:Fiducial_1mm_Mask2mm, symbol Mechanical:Fiducial
- added H1, H2, H3, H4: MountingHole_Pad, MountingHole:MountingHole_2.2mm_M2_Pad_Via, symbol Mechanical:MountingHole_Pad
Connections:
- net GND: now also H1.1, H2.1, H3.1, H4.1
Other:
- note added: "Fiducial Markers"
- note added: "Mounting Holes (M3)"
