File: Learn_KiCad.kicad_pcb (KiCad board)
At the start: 4 copper layers, 41 parts, among them J1 USB_C_Receptacle_USB2.0, J2 TC2030, J3 Conn_01x04_Pin, J4 Conn_Coaxial, SW1 SW_Push, U1 MIC5365-3.3YD5, U2 USBLC6-2SC6, U3 STM32WB55CEU6, X1 32kHz768, X2 32MHz

Commit message: 2024-01-09 22:03
Parts:
- moved U2 71.5 mm to (51.0, 70.0)
- moved J1 62.1 mm to (42.9, 69.7), turned to -90 degrees
- moved L2 59.3 mm to (70.0, 62.0)
- moved J2 56.0 mm to (59.5, 70.0), turned to -90 degrees
- moved L1 55.8 mm to (68.8, 64.0), turned to 90 degrees
- moved X2 51.8 mm to (75.5, 64.0), turned to 90 degrees
- moved R4 50.8 mm to (72.0, 76.5), turned to 90 degrees
- moved R5 50.6 mm to (73.0, 76.5), turned to 90 degrees
- moved C14 49.8 mm to (71.0, 64.0)
- moved J4 49.5 mm to (84.5, 68.8)
- moved X1 47.3 mm to (67.7, 76.0), turned to 180 degrees
- moved L3 46.9 mm to (78.0, 68.8)
- moved C18 45.8 mm to (65.5, 76.0), turned to -90 degrees
- moved J3 43.6 mm to (71.1, 79.3)
- moved FLT1 42.5 mm to (81.2, 68.8)
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
Commit message: 2024-01-13 22:28
Parts:
- moved R2 80.5 mm to (43.2, 63.5), turned to 180 degrees
- moved R1 74.5 mm to (43.2, 75.8), turned to 180 degrees
- moved U1 71.1 mm to (50.5, 76.0), turned to -90 degrees
- moved C1 60.4 mm to (50.5, 73.0), turned to 180 degrees
- moved C2 59.8 mm to (50.5, 79.0), turned to 180 degrees
- moved R6 58.5 mm to (64.0, 79.8)
- moved R7 57.8 mm to (64.8, 81.5), turned to -90 degrees
- moved C3 51.3 mm to (66.8, 62.2), turned to 180 degrees
- moved D1 50.8 mm to (76.2, 76.0), turned to 90 degrees
- moved C6 49.0 mm to (63.8, 75.8), turned to -90 degrees
- moved SW1 48.1 mm to (70.8, 81.2)
- moved C10 47.0 mm to (67.2, 63.5)
- moved C9 46.5 mm to (63.8, 73.0), turned to 90 degrees
- moved C19 46.0 mm to (63.5, 81.5), turned to -90 degrees
- moved C7 45.8 mm to (64.5, 69.2), turned to 180 degrees
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Connections:
- net Net-(R7-Pad2) renamed /BSW

Commit message: 2024-02-01 8:33am
Parts:
- added FM1: Fiducial, Fiducial:Fiducial_1mm_Mask2mm, F.Cu at (38.8, 60.8)
- added FM2: Fiducial, Fiducial:Fiducial_1mm_Mask2mm, F.Cu at (80.0, 62.8)
- added FM3: Fiducial, Fiducial:Fiducial_1mm_Mask2mm, F.Cu at (80.5, 83.5)
- added H1: MountingHole_Pad, MountingHole:MountingHole_2.2mm_M2_Pad_Via, F.Cu at (49.4, 62.5)
- added H2: MountingHole_Pad, MountingHole:MountingHole_2.2mm_M2_Pad_Via, F.Cu at (49.4, 83.6)
- added H3: MountingHole_Pad, MountingHole:MountingHole_2.2mm_M2_Pad_Via, F.Cu at (84.4, 62.6)
- added H4: MountingHole_Pad, MountingHole:MountingHole_2.2mm_M2_Pad_Via, F.Cu at (84.4, 83.5)
Routing:
- added copper zone on In1.Cu, net GND
- added copper zone on In2.Cu, net GND
Other:
- board outline added: 49 x 26 mm

Commit message: 2024-02-15 21:52
Parts:
- moved FM1 0.71 mm to (39.2, 61.2)
- moved C8 0.25 mm to (71.8, 75.5)
- moved C17 0.20 mm to (69.8, 76.0)
- turned C10 to 180 degrees
Routing:
- net GND: track 0.00 -> 10.5 mm, vias 0 -> 14
Changed lines of the file:
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@@
   )
   (footprint "Capacitor_SMD:C_0402_1005Metric" (layer "F.Cu")
-    (at 64.5 69.23 180)
+    (at 64.5 69.25 180)
     (descr "Capacitor SMD 0402 (1005 Metric), square (rectangular) end terminal, IPC_7351 nominal, (Body size source: IPC-SM-782 page 76, https://www.pcb-3d.com/wordpress/wp-content/uploads/ipc-sm-782a_amendment_1_and_2.pdf), generated with kicad-footprint-generator")
     (tags "capacitor")
@@
     (property "ki_keywords" "cap capacitor")
     (attr smd)
-    (fp_text reference "C7" (at 0 -1.16) (layer "F.SilkS")
+    (fp_text reference "C7" (at 0 0.98) (layer "F.SilkS")
         (effects (font (size 0.5 0.5) (thickness 0.125)))
     )
@@
   )
   (footprint "Capacitor_SMD:C_0402_1005Metric" (layer "F.Cu")
-    (at 65.3 76 -90)
+    (at 65.25 76 -90)
     (descr "Capacitor SMD 0402 (1005 Metric), square (rectangular) end terminal, IPC_7351 nominal, (Body size source: IPC-SM-782 page 76, https://www.pcb-3d.com/wordpress/wp-content/uploads/ipc-sm-782a_amendment_1_and_2.pdf), generated with kicad-footprint-generator")
     (tags "capacitor")
@@
   )
   (footprint "Capacitor_SMD:C_0402_1005Metric" (layer "F.Cu")
-    (at 67.25 63.5)
+    (at 67.25 63.5 180)
     (descr "Capacitor SMD 0402 (1005 Metric), square (rectangular) end terminal, IPC_7351 nominal, (Body size source: IPC-SM-782 page 76, https://www.pcb-3d.com/wordpress/wp-content/uploads/ipc-sm-782a_amendment_1_and_2.pdf), generated with kicad-footprint-generator")
     (tags "capacitor")
@@
     (property "ki_keywords" "cap capacitor")
     (attr smd)
-    (fp_text reference "C10" (at 0 -1) (layer "F.SilkS")
+    (fp_text reference "C10" (at 1.77 0) (layer "F.SilkS")
         (effects (font (size 0.5 0.5) (thickness 0.125)))
     )
@@
     (fp_line (start 0.5 0.25) (end -0.5 0.25)
       (stroke (width 0.1) (type solid)) (layer "F.Fab"))
-    (pad "1" smd roundrect (at -0.48 0) (size 0.56 0.62) (layers "F.Cu" "F.Paste" "F.Mask") (roundrect_rratio 0.25)
+    (pad "1" smd roundrect (at -0.48 0 180) (size 0.56 0.62) (layers "F.Cu" "F.Paste" "F.Mask") (roundrect_rratio 0.25)
       (net 3 "+3.3V") (pintype "passive"))
-    (pad "2" smd roundrect (at 0.48 0) (size 0.56 0.62) (layers "F.Cu" "F.Paste" "F.Mask") (roundrect_rratio 0.25)
+    (pad "2" smd roundrect (at 0.48 0 180) (size 0.56 0.62) (layers "F.Cu" "F.Paste" "F.Mask") (roundrect_rratio 0.25)
       (net 2 "GND") (pintype "passive"))
     (model "${KICAD6_3DMODEL_DIR}/Capacitor_SMD.3dshapes/C_0402_1005Metric.wrl"
@@
     (property "ki_keywords" "inductor choke coil reactor magnetic")
     (attr smd)
-    (fp_text reference "L1" (at 0.5 -1 90) (layer "F.SilkS")
+    (fp_text reference "L1" (at -1.25 0 90) (layer "F.SilkS")
         (effects (font (size 0.5 0.5) (thickness 0.125)))
     )
@@
     (property "ki_keywords" "cap capacitor")
     (attr smd)
-    (fp_text reference "C9" (at 1.48 0 90) (layer "F.SilkS")
+    (fp_text reference "C9" (at 2.23 0 90) (layer "F.SilkS")
         (effects (font (size 0.5 0.5) (thickness 0.125)))
     )
@@
   )
   (footprint "Capacitor_SMD:C_0402_1005Metric" (layer "F.Cu")
-    (at 69.55 75.98 -90)
+    (at 69.75 76 -90)
     (descr "Capacitor SMD 0402 (1005 Metric), square (rectangular) end terminal, IPC_7351 nominal, (Body size source: IPC-SM-782 page 76, https://www.pcb-3d.com/wordpress/wp-content/uploads/ipc-sm-782a_amendment_1_and_2.pdf), generated with kicad-footprint-generator")
     (tags "capacitor")
@@
   )
   (footprint "Capacitor_SMD:C_0402_1005Metric" (layer "F.Cu")
-    (at 72 75.5)
+    (at 71.75 75.5)
     (descr "Capacitor SMD 0402 (1005 Metric), square (rectangular) end terminal, IPC_7351 nominal, (Body size source: IPC-SM-782 page 76, https://www.pcb-3d.com/wordpress/wp-content/uploads/ipc-sm-782a_amendment_1_and_2.pdf), generated with kicad-footprint-generator")
     (tags "capacitor")
@@
   )
   (footprint "Fiducial:Fiducial_1mm_Mask2mm" (layer "F.Cu")
-    (at 38.75 60.75)
+    (at 39.25 61.25)
     (descr "Circular Fiducial, 1mm bare copper, 2mm soldermask opening (Level A)")
     (tags "fiducial")
@@
   (gr_line (start 87 86) (end 38 86)
     (stroke (width 0.1) (type default)) (layer "Edge.Cuts"))
+  (segment (start 64.02 69.27) (end 64 69.25) (width 0.5) (layer "F.Cu") (net 2))
+  (segment (start 66.625 63.5) (end 65.875 63.5) (width 0.5) (layer "F.Cu") (net 2))
+  (segment (start 76.5 69.875) (end 76.5 70.625) (width 0.5) (layer "F.Cu") (net 2))
+  (segment (start 79.5 69.875) (end 79.5 70.625) (width 0.5) (layer "F.Cu") (net 2))
+  (segment (start 64 68.54) (end 64 69.25) (width 0.5) (layer "F.Cu") (net 2))
+  (segment (start 74.75 70.625) (end 74.75 71.375) (width 0.5) (layer "F.Cu") (net 2))
+  (segment (start 63.5 82.125) (end 63.5 82.875) (width 0.5) (layer "F.Cu") (net 2))
+  (segment (start 63.75 72.5) (end 63.75 71.75) (width 0.5) (layer "F.Cu") (net 2))
+  (segment (start 69.75 76.5) (end 69.75 77.25) (width 0.5) (layer "F.Cu") (net 2))
+  (segment (start 74.875 68) (end 75.625 68) (width 0.5) (layer "F.Cu") (net 2))
+  (segment (start 64.75 72.5) (end 64.75 71.75) (width 0.5) (layer "F.Cu") (net 2))
+  (segment (start 64.125 78) (end 64.875 78) (width 0.5) (layer "F.Cu") (net 2))
+  (segment (start 66.75 64.5) (end 66 64.5) (width 0.5) (layer "F.Cu") (net 2))
+  (segment (start 65.25 76.5) (end 65.25 77.25) (width 0.5) (layer "F.Cu") (net 2))
+  (segment (start 72.25 75.5) (end 72.25 76.25) (width 0.5) (layer "F.Cu") (net 2))
+  (via (at 64.75 71.75) (size 0.7) (drill 0.3) (layers "F.Cu" "B.Cu") (free) (net 2))
+  (via (at 76.5 70.625) (size 0.7) (drill 0.3) (layers "F.Cu" "B.Cu") (free) (net 2))
+  (via (at 66 64.5) (size 0.7) (drill 0.3) (layers "F.Cu" "B.Cu") (free) (net 2))
+  (via (at 75.625 68) (size 0.7) (drill 0.3) (layers "F.Cu" "B.Cu") (free) (net 2))
+  (via (at 69.75 77.25) (size 0.7) (drill 0.3) (layers "F.Cu" "B.Cu") (free) (net 2))
+  (via (at 65.875 63.5) (size 0.7) (drill 0.3) (layers "F.Cu" "B.Cu") (free) (net 2))
+  (via (at 79.5 70.625) (size 0.7) (drill 0.3) (layers "F.Cu" "B.Cu") (free) (net 2))
+  (via (at 63.5 82.875) (size 0.7) (drill 0.3) (layers "F.Cu" "B.Cu") (free) (net 2))
+  (via (at 65.25 77.25) (size 0.7) (drill 0.3) (layers "F.Cu" "B.Cu") (free) (net 2))
+  (via (at 64.875 78) (size 0.7) (drill 0.3) (layers "F.Cu" "B.Cu") (free) (net 2))
+  (via (at 74.75 71.375) (size 0.7) (drill 0.3) (layers "F.Cu" "B.Cu") (free) (net 2))
+  (via (at 63.75 71.75) (size 0.7) (drill 0.3) (layers "F.Cu" "B.Cu") (free) (net 2))
+  (via (at 72.25 76.25) (size 0.7) (drill 0.3) (layers "F.Cu" "B.Cu") (free) (net 2))
+  (via (at 64 68.54) (size 0.7) (drill 0.3) (layers "F.Cu" "B.Cu") (free) (net 2))
   (zone (net 2) (net_name "GND") (layers "In1.Cu" "In2.Cu") (hatch edge 0.5)
     (connect_pads (clearance 0.3))
     (min_thickness 0.15) (filled_areas_thickness no)
+    (fill yes (thermal_gap 0.4) (thermal_bridge_width 0.25))
+    (polygon
+      (pts
+        (xy 38 60)
+        (xy 87 60)
+        (xy 87 86)
+        (xy 38 86)
+      )
+    )
+  )
+  (zone (net 2) (net_name "GND") (layers "In1.Cu" "In2.Cu") (hatch edge 0.5)
+    (priority 1)
+    (connect_pads (clearance 0.3))
+    (min_thickness 0.15) (filled_areas_thickness no)

Commit message: 2024-03-16 14:17
Parts:
- moved R3 0.10 mm to (77.5, 76.0)
- turned C13 to 180 degrees
Routing:
- net /RF: track 0.00 -> 4.13 mm
- net GND: track 10.5 -> 13.5 mm, vias 14 -> 54
- net +3.3V: track 0.00 -> 2.25 mm, vias 0 -> 11
- net /RF_MATCH: track 0.00 -> 2.15 mm
- net /RF_ANT: track 0.00 -> 1.59 mm
- net +5V: vias 0 -> 1

Commit message: 2024-04-07 13:56
Parts:
- moved C19 10.9 mm to (74.2, 83.2)
- moved R6 9.62 mm to (73.5, 81.2), turned to 180 degrees
- moved R7 8.42 mm to (73.0, 83.2)
- moved C2 3.89 mm to (53.2, 76.2), turned to 90 degrees
- moved SW1 3.81 mm to (67.2, 82.8), turned to 180 degrees
- moved C17 1.31 mm to (68.8, 75.2), turned to 0 degrees
- moved C18 1.25 mm to (66.2, 75.2), turned to 180 degrees
- moved C5 0.82 mm to (75.5, 67.2)
- moved X1 0.75 mm to (67.5, 76.8)
- moved C7 0.56 mm to (64.2, 68.8)
- moved X2 0.50 mm to (75.5, 63.5)
- moved C6 0.25 mm to (63.8, 75.5)
- moved C13 0.15 mm to (63.8, 78.0), turned to 90 degrees
Routing:
- net Net-(J3-Pin_3): track 0.00 -> 34.2 mm
- net Net-(J3-Pin_2): track 0.00 -> 33.0 mm
- net /SWD_NRST: track 0.00 -> 32.3 mm
- net /USB_D+: track 0.00 -> 22.6 mm
- net +5V: track 0.00 -> 21.7 mm, vias 1 -> 0
- net /USB_D-: track 0.00 -> 21.3 mm
- net +3.3V: track 2.25 -> 21.6 mm, vias 11 -> 12
- net /BOOT0: track 0.00 -> 14.9 mm, vias 0 -> 2
- net GND: track 13.5 -> 25.2 mm, vias 54 -> 110
- net /SWD_DIO: track 0.00 -> 11.4 mm
- net /SWD_CLK: track 0.00 -> 8.70 mm
- net /SWD_TRC: track 0.00 -> 8.55 mm
- net /USBC_D-: track 0.00 -> 6.41 mm
- net /USBC_CC1: track 0.00 -> 6.17 mm
- net /LED_A: track 0.00 -> 6.11 mm
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- added copper zone on F.Cu, net +3.3V
- added copper zone on F.Cu, net /SMPSFB
- added copper zone on F.Cu, net GND
Other:
- board text added: "H2"
